File: hardware/eagle_files/RF433Shield/rf433schield.sch (EAGLE design)
At the start: 2 parts, among them U1 ARDUINOR3-DIMENSION

Commit message: New version
Parts:
- added U$2: ICEEPOT_LOGO, RFM:ICEEPOT_LOGO
Changed lines of the file:
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@@
 <part name="U$1" library="RFM" deviceset="RF-LINK_RX" device=""/>
 <part name="U1" library="RFM" deviceset="ARDUINOR3" device="-DIMENSION"/>
+<part name="U$2" library="RFM" deviceset="ICEEPOT_LOGO" device=""/>
 </parts>
 <sheets>
@@
 <instance part="U$1" gate="G$1" x="91.44" y="55.88"/>
 <instance part="U1" gate="G$1" x="25.4" y="53.34"/>
+<instance part="U$2" gate="G$1" x="73.66" y="71.12"/>
 </instances>
 <busses>
@@
 </sheet>
 </sheets>
+<errors>
+</errors>
 </schematic>
 </drawing>
